File: js220_fp_template.kicad_pcb (KiCad board)
At the start: 2 copper layers, 95 x 24.7 mm, 5 parts, among them J1 JS220

Commit message: Fixed flipped pinout with I+ I-
Connections:
- J1 pad 1: /I- -> /I+
- J1 pad 2: /I- -> /I+
- J1 pad 3: I+ -> /I-
- J1 pad 4: I+ -> /I-
Changed lines of the file:
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@@
   (title_block
     (title "Joulescope JS220 Front Panel Template")
-    (date "2022-10-23")
-    (rev "1.1")
+    (date "2022-11-12")
+    (rev "1.2")
     (company "Alvaro Prieto")
   )
@@
   (net 1 "/V+")
   (net 2 "/V-")
-  (net 3 "I+")
+  (net 3 "/I+")
   (net 4 "/I-")
   (net 5 "/CH_GND")
   (footprint "Joulescope:MOUNTING_HOLE_3.3MM" locked (layer "F.Cu")
     (at 130.95 100)
-    (property "Sheetfile" "File: js220_fp_template.kicad_sch")
+    (property "Sheetfile" "js220_fp_template.kicad_sch")
     (property "Sheetname" "")
     (attr smd)
@@
   (footprint "Joulescope:MOUNTING_HOLE_3.5_W_KO" locked (layer "F.Cu")
     (at 193.71 100)
-    (property "Sheetfile" "File: js220_fp_template.kicad_sch")
+    (property "Sheetfile" "js220_fp_template.kicad_sch")
     (property "Sheetname" "")
     (attr smd)
@@
   (footprint "Joulescope:MOUNTING_HOLE_3.5_W_KO" locked (layer "F.Cu")
     (at 106.29 100)
-    (property "Sheetfile" "File: js220_fp_template.kicad_sch")
+    (property "Sheetfile" "js220_fp_template.kicad_sch")
     (property "Sheetname" "")
     (attr smd)
@@
   (footprint "Joulescope:TINY_TP" locked (layer "F.Cu")
     (at 169.6 89.5)
-    (property "Sheetfile" "File: js220_fp_template.kicad_sch")
+    (property "Sheetfile" "js220_fp_template.kicad_sch")
     (property "Sheetname" "")
     (attr smd)
@@
   (footprint "Joulescope:SAMTEC_TSM-103-01-S-DV-A" locked (layer "B.Cu")
     (at 150 101.29)
-    (property "Sheetfile" "File: js220_fp_template.kicad_sch")
+    (property "Sheetfile" "js220_fp_template.kicad_sch")
     (property "Sheetname" "")
     (attr through_hole)
@@
     (pad "" np_thru_hole circle locked (at -1.27 0) (size 1.73 1.73) (drill 1.73) (layers *.Cu *.Mask))
     (pad "1" smd custom locked (at 2.54 2.475) (size 0.8 2.5) (layers "B.Cu")
-      (net 4 "/I-") (pinfunction "I-") (pintype "power_out") (zone_connect 0)
+      (net 3 "/I+") (pinfunction "I+") (pintype "power_in") (zone_connect 0)
       (options (clearance outline) (anchor rect))
       (primitives
@@
       ))
     (pad "2" smd custom locked (at 2.54 -2.475) (size 0.8 2.5) (layers "B.Cu")
-      (net 4 "/I-") (pinfunction "I-") (pintype "power_out") (zone_connect 0)
+      (net 3 "/I+") (pinfunction "I+") (pintype "passive") (zone_connect 0)
       (options (clearance outline) (anchor rect))
       (primitives
@@
       ))
     (pad "3" smd custom locked (at 0 2.475) (size 0.8 2.5) (layers "B.Cu")
-      (net 3 "I+") (pinfunction "I+") (pintype "power_in") (zone_connect 0)
+      (net 4 "/I-") (pinfunction "I-") (pintype "power_out") (zone_connect 0)
       (options (clearance outline) (anchor rect))
       (primitives
@@
       ))
     (pad "4" smd custom locked (at 0 -2.475) (size 0.8 2.5) (layers "B.Cu")
-      (net 3 "I+") (pinfunction "I+") (pintype "power_in") (zone_connect 0)
+      (net 4 "/I-") (pinfunction "I-") (pintype "passive") (zone_connect 0)
       (options (clearance outline) (anchor rect))
       (primitives
